File: PCB/Controllers/EC_Pro2_Controller_Lite/EC_Pro2_Controller_Lite.kicad_sch (KiCad schematic)
At the start: 8 parts, among them J1 JST, U1 SRV05-4

Commit message: Updated sheets
Other:
- company: Cipulot PCB Design -> LU.SV Solutions
