File: PCB/EC_Pro2_Mainboard/analog.kicad_sch (KiCad schematic)
At the start: 25 parts, among them U3 74HC4051, U4 OPA350, U5 74HC4051

Commit message: Updated sheets
Other:
- company: Cipulot PCB Design  -> LU.SV Solutions
