File: PCB/Controllers/EC_Pro2_Controller_Normal/EC_Pro2_Controller_Normal.kicad_pcb (KiCad board)
At the start: 2 copper layers, 141.5 x 36 mm, 51 parts, among them J1 JST, J2 USB_A, J3 USB_A, U1 MIC2026-2BM, U2 SRV05-4, U3 SRV05-4, U4 SRV05-4, U5 FE1.1, Y1 12MHz

Commit message: Replaced type A port to USB1130-15-A
Parts:
- removed Je: USB_A, cipulot_parts:USB-SMT-04F-S1-B1-R9A
- added J4: USB_A, USB1130-15-A:GCT_USB1130-15-A_REVA, F.Cu at (155.1, 66.3)
- J2, J3: footprint cipulot_parts:USB-SMT-04F-S1-B1-R9A -> USB1130-15-A:GCT_USB1130-15-A_REVA
- moved J3 3.42 mm to (127.7, 66.3), turned to 180 degrees
- moved J2 3.42 mm to (53.9, 66.0), turned to 0 degrees
Connections:
- J1 pad : GND -> (no net)
Routing:
- net /PORT2_PWR: track 40.5 -> 44.0 mm
- net /PORT1_PWR: track 22.0 -> 25.2 mm
- net GNDPWR: track 293.7 -> 290.7 mm
- net D1+: track 35.8 -> 38.2 mm
- net D1-: track 35.8 -> 38.2 mm
- net D2-: track 64.8 -> 67.2 mm
- net D2+: track 64.7 -> 67.1 mm
- net VCC: track 146.8 -> 144.7 mm
- net D3-: track 63.8 -> 61.9 mm
- net D3+: track 63.8 -> 62.0 mm
- net GND: vias 73 -> 71
Other:
- board text added: "EC Pro2 Controller-Normal by Cipulot Modified for USB1130-15-A USB Port https://github.com/Armastardo/EC-Pro-2"
