File: PCB/Controllers/EC_Pro2_Controller_Normal/EC_Pro2_Controller_Normal.kicad_sch (KiCad schematic)
At the start: 49 parts, among them J1 JST, J2 USB_A, J3 USB_A, J4 USB_A, U1 MIC2026-2BM, U2 SRV05-4, U3 SRV05-4, U4 SRV05-4, U5 FE1.1, Y1 12MHz

Commit message: Updated sheets
Other:
- company: Cipulot PCB Design -> LU.SV Solutions

Commit message: Replaced type A port to USB1130-15-A
Parts:
- J2, J3, J4: footprint cipulot_parts:USB-SMT-04F-S1-B1-R9A -> USB1130-15-A:GCT_USB1130-15-A_REVA; LCSC C718022 -> (none)
Changed lines of the file:
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@@
 			)
 		)
-		(property "Footprint" "cipulot_parts:USB-SMT-04F-S1-B1-R9A"
+		(property "Footprint" "USB1130-15-A:GCT_USB1130-15-A_REVA"
 			(at 78.105 151.765 0)
 			(effects
@@
 			)
 		)
-		(property "LCSC" "C718022"
-			(at 74.295 150.495 0)
-			(effects
-				(font
-					(size 1.27 1.27)
-				)
-				(hide yes)
-			)
-		)
 		(pin "1"
 		)
@@
 			)
 		)
-		(property "Footprint" "cipulot_parts:USB-SMT-04F-S1-B1-R9A"
+		(property "Footprint" "USB1130-15-A:GCT_USB1130-15-A_REVA"
 			(at 113.03 133.985 0)
 			(effects
@@
 			)
 		)
-		(property "LCSC" "C718022"
-			(at 109.22 132.715 0)
-			(effects
-				(font
-					(size 1.27 1.27)
-				)
-				(hide yes)
-			)
-		)
 		(pin "1"
 		)
@@
 			)
 		)
-		(property "Footprint" "cipulot_parts:USB-SMT-04F-S1-B1-R9A"
+		(property "Footprint" "USB1130-15-A:GCT_USB1130-15-A_REVA"
 			(at 33.655 151.765 0)
 			(effects
@@
 			(at 29.845 150.495 0)
 			(effects
-				(font
-					(size 1.27 1.27)
-				)
-				(hide yes)
-			)
-		)
-		(property "LCSC" "C718022"
-			(at 29.845 150.495 0)
-			(effects
